File: kicad/A603EP_Mouse.kicad_pcb (KiCad board)
At the start: 2 copper layers, 38.9 x 66.4 mm, 18 parts, among them J1 USB cable, SW1 Left click, SW2 Right click, SW3 Middle click, SW4 Side button 1, SW5 Side button 2, SW6 DPI (K6), U1 A603EP

Commit message: fix: updating pcb and pretty files wrt to notch for mouse encoder identified during path tracing and design error checker
Routing:
- net +5V: track 0.00 -> 150.8 mm, vias 0 -> 4
- net BL_K: track 0.00 -> 147.1 mm
- net S1: track 0.00 -> 126.3 mm
- net R0: track 0.00 -> 86.2 mm
- net R1: track 0.00 -> 59.4 mm
- net R2: track 0.00 -> 49.9 mm
- net ZA: track 0.00 -> 42.6 mm
- net ZB: track 0.00 -> 39.1 mm
- net USB_DM: track 0.00 -> 28.5 mm
- net USB_DP: track 0.00 -> 23.0 mm
- net GND: track 0.00 -> 22.7 mm
- net LED_DRV: track 0.00 -> 14.1 mm
- net BL_DRV: track 0.00 -> 12.4 mm
- net LED_K: track 0.00 -> 5.81 mm
- added copper zone on B.Cu, net GND
- added copper zone on F.Cu, net GND
Other:
- outline, holes or cut-outs redrawn
